File: hardware/media-controller.kicad_sch (KiCad schematic)
At the start: 43 parts, among them J1 USB_C_Receptacle_USB2.0_14P, SW1 RotaryEncoder_Switch, SW2 MX Style Switch, SW3 MX Style Switch, SW4 MX Style Switch, SW5 RUN, SW6 USB_BOOT, U1 RP2040, U2 XC6206P332MR-G, U3 W25Q16JVSS, U4 ER_OLEDM0.91_1x-I2C, Y1 ABM8-272-T3

Commit message: Updated schematic.
Other:
- note added: "0.91"I2C SSD1306 OLED Display"
Changed lines of the file:
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@@
+		)
+	)
+	(text "0.91\"I2C SSD1306 OLED Display "
+		(exclude_from_sim no)
+		(at 153.67 161.036 0)
+		(effects
+			(font
+				(size 1.778 1.778)
+			)
 		)
 	)

Commit message: Updated schematic and models.
Parts:
- removed J1: USB_C_Receptacle_USB2.0_14P, symbol Connector:USB_C_Receptacle_USB2.0_14P
- added J1: XKB Connection U262-161N-4BVC11, Connector_USB:USB_C_Receptacle_XKB_U262-16XN-4BVC11, symbol Connector:USB_C_Receptacle_USB2.0_16P
- SW1: value RotaryEncoder_Switch -> PEC12R-4215F-S0024; footprint (none) -> Custom_Parts:PEC12R-4215F-S0024
- SW5, SW6: footprint (none) -> Button_Switch_SMD:SW_SPST_TS-1088-xR025
Connections:
- net +5V: now also J1.A4 (VBUS), J1.A9 (VBUS), J1.B4 (VBUS), J1.B9 (VBUS)
- net D+: now also J1.A6 (D+), J1.B6 (D+)
- net D-: now also J1.A7 (D-), J1.B7 (D-)
- net GND: now also J1.A1 (GND), J1.A12 (GND), J1.B1 (GND), J1.B12 (GND), J1.SH (SHIELD)
- net at R2.1: now also J1.A5 (CC1)
- net at R1.1: now also J1.B5 (CC2)
- no-connect marks 24 -> 26
Changed lines of the file:
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@@
 	)
 	(no_connect
+		(at 157.48 55.88)
+	)
+	(no_connect
 		(at 99.06 105.41)
 	)
@@
 	)
 	(no_connect
+		(at 157.48 53.34)
+	)
+	(no_connect
 		(at 99.06 90.17)
 	)
@@
 			)
 		)
-		(property "Footprint" ""
+		(property "Footprint" "Button_Switch_SMD:SW_SPST_TS-1088-xR025"
 			(at 35.56 57.15 0)
 			(hide yes)
@@
 			)
 		)
-		(property "Value" "RotaryEncoder_Switch"
+		(property "Value" "PEC12R-4215F-S0024"
 			(at 237.49 88.9 0)
 			(show_name no)
@@
 			)
 		)
-		(property "Footprint" ""
+		(property "Footprint" "Custom_Parts:PEC12R-4215F-S0024"
 			(at 233.68 92.456 0)
 			(hide yes)
@@
 	)
 	(symbol
+		(lib_id "Connector:USB_C_Receptacle_USB2.0_16P")
+		(at 142.24 40.64 0)
+		(unit 1)
+		(body_style 1)
+		(exclude_from_sim no)
+		(in_bom yes)
+		(on_board yes)
+		(in_pos_files yes)
+		(dnp no)
+		(fields_autoplaced yes)
+		(property "Reference" "J1"
+			(at 142.24 17.78 0)
+			(show_name no)
+			(do_not_autoplace no)
+			(effects
+				(font
+					(size 1.27 1.27)
+				)
+			)
+		)
+		(property "Value" "XKB Connection U262-161N-4BVC11"
+			(at 142.24 20.32 0)
+			(show_name no)
+			(do_not_autoplace no)
+			(effects
+				(font
+					(size 1.143 1.143)
+				)
+			)
+		)
+		(property "Footprint" "Connector_USB:USB_C_Receptacle_XKB_U262-16XN-4BVC11"
+			(at 146.05 40.64 0)
+			(hide yes)
+			(show_name no)
+			(do_not_autoplace no)
+			(effects
+				(font
+					(size 1.27 1.27)
+				)
+			)
+		)
+		(property "Datasheet" "https://www.usb.org/sites/default/files/documents/usb_type-c.zip"
+			(at 146.05 40.64 0)
+			(hide yes)
+			(show_name no)
+			(do_not_autoplace no)
+			(effects
+				(font
+					(size 1.27 1.27)
+				)
+			)
+		)
+		(property "Description" "USB 2.0-only 16P Type-C Receptacle connector"
+			(at 142.24 40.64 0)
+			(hide yes)
+			(show_name no)
+			(do_not_autoplace no)
+			(effects
+				(font
+					(size 1.27 1.27)
+				)
+			)
+		)
+		(pin "B12"
+		)
+		(pin "B6"
+		)
+		(pin "A12"
+		)
+		(pin "B8"
+		)
+		(pin "A5"
+		)
+		(pin "A1"
+		)
+		(pin "B9"
+		)
+		(pin "B5"
+		)
+		(pin "B7"
+		)
+		(pin "A7"
+		)
+		(pin "A9"
+		)
+		(pin "A6"
+		)
+		(pin "B4"
+		)
+		(pin "SH"
+		)
+		(pin "A4"
+		)
+		(pin "A8"
+		)
+		(pin "B1"
+		)
+		(instances
+			(project "media-controller"
+				(path "/26b913e7-2823-4a13-b717-dd54292058d7"
+					(reference "J1")
+					(unit 1)
+				)
+			)
+		)
+	)
+	(symbol
 		(lib_id "power:GND")
 		(at 135.89 102.87 0)
@@
 			)
 		)
-		(property "Footprint" ""
+		(property "Footprint" "Button_Switch_SMD:SW_SPST_TS-1088-xR025"
 			(at 195.58 43.18 0)
 			(hide yes)
@@
 					(unit 1)
 				)
-			)
-		)
-	)
-	(symbol
-		(lib_id "Connector:USB_C_Receptacle_USB2.0_14P")
-		(at 142.24 40.64 0)
-		(unit 1)
-		(body_style 1)
-		(exclude_from_sim no)
-		(in_bom yes)
-		(on_board yes)
-		(in_pos_files yes)
-		(dnp no)
-		(fields_autoplaced yes)
-		(property "Reference" "J1"
-			(at 142.24 17.78 0)
-			(show_name no)
-			(do_not_autoplace no)
-			(effects
-				(font
-					(size 1.27 1.27)
-				)
-			)
-		)
-		(property "Value" "USB_C_Receptacle_USB2.0_14P"
-			(at 142.24 20.32 0)
-			(show_name no)
-			(do_not_autoplace no)
-			(effects
-				(font
-					(size 1.27 1.27)
-				)
-			)
-		)
-		(property "Footprint" ""
-			(at 146.05 40.64 0)
-			(hide yes)
-			(show_name no)
-			(do_not_autoplace no)
-			(effects
-				(font
-					(size 1.27 1.27)
-				)
-			)
-		)
-		(property "Datasheet" "https://www.usb.org/sites/default/files/documents/usb_type-c.zip"
-			(at 146.05 40.64 0)
-			(hide yes)
-			(show_name no)
-			(do_not_autoplace no)
-			(effects
-				(font
-					(size 1.27 1.27)
-				)
-			)
-		)
-		(property "Description" "USB 2.0-only 14P Type-C Receptacle connector"
-			(at 142.24 40.64 0)
-			(hide yes)
-			(show_name no)
-			(do_not_autoplace no)
-			(effects
-				(font
-					(size 1.27 1.27)
-				)
-			)
-		)
-		(pin "B5"
-		)
-		(pin "B4"
-		)
-		(pin "B1"
-		)
-		(pin "A12"
-		)
-		(pin "A9"
-		)
-		(pin "A7"
-		)
-		(pin "A6"
-		)
-		(pin "A5"
-		)
-		(pin "A1"
-		)
-		(pin "A4"
-		)
-		(pin "B7"
-		)
-		(pin "B12"
-		)
-		(pin "B6"
-		)
-		(pin "B9"
-		)
-		(pin "SH"
-		)
-		(instances
-			(project "media-controller"
-				(path "/26b913e7-2823-4a13-b717-dd54292058d7"
-					(reference "J1")
-					(unit 1)
-				)

Commit message: Updated schematic & footprints
Parts:
- C1, C2: footprint (none) -> Capacitor_SMD:C_0402_1005Metric_Pad0.74x0.62mm_HandSolder; Note (none) -> 15pF 50V C0G ±5% 0402
- C10, C11, C12, C13, C14, C15, C16, C17, C18, C19, C20, C21, C22, C23, C24, C6, C9: footprint (none) -> Capacitor_SMD:C_0402_1005Metric_Pad0.74x0.62mm_HandSolder
- C3, C4, C5, C7, C8: footprint (none) -> Capacitor_SMD:C_0805_2012Metric_Pad1.18x1.45mm_HandSolder
- R1, R2, R3, R4, R5, R6: footprint (none) -> Resistor_SMD:R_0603_1608Metric_Pad0.98x0.95mm_HandSolder
Other:
- note added: "50V C0G ±5% 0402"
- moved on the sheet: SW2, SW3, SW4

Commit message: Updated PCB.
Parts:
- C8: footprint Capacitor_SMD:C_0805_2012Metric_Pad1.18x1.45mm_HandSolder -> Capacitor_SMD:C_0603_1608Metric_Pad1.08x0.95mm_HandSolder
Changed lines of the file:
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@@
 			)
 		)
-		(property "Footprint" "Capacitor_SMD:C_0805_2012Metric_Pad1.18x1.45mm_HandSolder"
+		(property "Footprint" "Capacitor_SMD:C_0603_1608Metric_Pad1.08x0.95mm_HandSolder"
 			(at 25.0952 36.83 0)
 			(hide yes)
